File: subsheet/ESP32-C3-core.kicad_sch (KiCad schematic)
At the start: 14 parts, among them Q701 40MHz, U702 ESP32-C3

Commit message: Uknown changes?File formats?
Parts:
- renumbered C709 to C701, C710 to C702, C701 to C703, C702 to C704, C703 to C705, C704 to C706, C705 to C707, C706 to C708, C707 to C709, C708 to C710, U702 to U701
Changed lines of the file:
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@@
 		(on_board yes)
 		(dnp no)
-		(property "Reference" "C710"
+		(property "Reference" "C702"
 			(at 62.484 147.955 0)
 			(effects
@@
 			(project "ESP_bare_chip_test_board"
 				(path "/45b6f84a-e69b-48be-a49b-bc68872e2c15/01bb46e3-d129-4909-82a1-6bb013dc8f71/9be7d96f-e7c5-43f0-93fa-5964acc52bec"
-					(reference "C710")
+					(reference "C702")
 					(unit 1)
 				)
@@
 		(dnp no)
 		(fields_autoplaced yes)
-		(property "Reference" "C705"
+		(property "Reference" "C707"
 			(at 127 49.5363 0)
 			(effects
@@
 			(project "ESP_bare_chip_test_board"
 				(path "/45b6f84a-e69b-48be-a49b-bc68872e2c15/01bb46e3-d129-4909-82a1-6bb013dc8f71/9be7d96f-e7c5-43f0-93fa-5964acc52bec"
-					(reference "C705")
+					(reference "C707")
 					(unit 1)
 				)
@@
 		(dnp no)
 		(fields_autoplaced yes)
-		(property "Reference" "U702"
+		(property "Reference" "U701"
 			(at 141.8941 160.02 0)
 			(effects
@@
 			(project "ESP_bare_chip_test_board"
 				(path "/45b6f84a-e69b-48be-a49b-bc68872e2c15/01bb46e3-d129-4909-82a1-6bb013dc8f71/9be7d96f-e7c5-43f0-93fa-5964acc52bec"
-					(reference "U702")
+					(reference "U701")
 					(unit 1)
 				)
@@
 		(dnp no)
 		(fields_autoplaced yes)
-		(property "Reference" "C703"
+		(property "Reference" "C705"
 			(at 114.3 49.5363 0)
 			(effects
@@
 			(project "ESP_bare_chip_test_board"
 				(path "/45b6f84a-e69b-48be-a49b-bc68872e2c15/01bb46e3-d129-4909-82a1-6bb013dc8f71/9be7d96f-e7c5-43f0-93fa-5964acc52bec"
-					(reference "C703")
+					(reference "C705")
 					(unit 1)
 				)
@@
 		(dnp no)
 		(fields_autoplaced yes)
-		(property "Reference" "C707"
+		(property "Reference" "C709"
 			(at 162.56 62.2363 0)
 			(effects
@@
 			(project "ESP_bare_chip_test_board"
 				(path "/45b6f84a-e69b-48be-a49b-bc68872e2c15/01bb46e3-d129-4909-82a1-6bb013dc8f71/9be7d96f-e7c5-43f0-93fa-5964acc52bec"
-					(reference "C707")
+					(reference "C709")
 					(unit 1)
 				)
@@
 		(dnp no)
 		(fields_autoplaced yes)
-		(property "Reference" "#PWR0708"
+		(property "Reference" "#PWR0709"
 			(at 160.02 90.17 0)
 			(effects
@@
 			(project "ESP_bare_chip_test_board"
 				(path "/45b6f84a-e69b-48be-a49b-bc68872e2c15/01bb46e3-d129-4909-82a1-6bb013dc8f71/9be7d96f-e7c5-43f0-93fa-5964acc52bec"
-					(reference "#PWR0708")
+					(reference "#PWR0709")
 					(unit 1)
 				)
@@
 		(dnp no)
 		(fields_autoplaced yes)
-		(property "Reference" "C701"
+		(property "Reference" "C703"
 			(at 81.28 69.8563 0)
 			(effects
@@
 			(project "ESP_bare_chip_test_board"
 				(path "/45b6f84a-e69b-48be-a49b-bc68872e2c15/01bb46e3-d129-4909-82a1-6bb013dc8f71/9be7d96f-e7c5-43f0-93fa-5964acc52bec"
-					(reference "C701")
+					(reference "C703")
 					(unit 1)
 				)
@@
 		(dnp no)
 		(fields_autoplaced yes)
-		(property "Reference" "#PWR0709"
+		(property "Reference" "#PWR0710"
 			(at 167.64 196.85 0)
 			(effects
@@
 			(project "ESP_bare_chip_test_board"
 				(path "/45b6f84a-e69b-48be-a49b-bc68872e2c15/01bb46e3-d129-4909-82a1-6bb013dc8f71/9be7d96f-e7c5-43f0-93fa-5964acc52bec"
-					(reference "#PWR0709")
+					(reference "#PWR0710")
 					(unit 1)
 				)
@@
 		(dnp no)
 		(fields_autoplaced yes)
-		(property "Reference" "#PWR0707"
+		(property "Reference" "#PWR0708"
 			(at 160.02 72.39 0)
 			(effects
@@
 			(project "ESP_bare_chip_test_board"
 				(path "/45b6f84a-e69b-48be-a49b-bc68872e2c15/01bb46e3-d129-4909-82a1-6bb013dc8f71/9be7d96f-e7c5-43f0-93fa-5964acc52bec"
-					(reference "#PWR0707")
+					(reference "#PWR0708")
 					(unit 1)
 				)
@@
 		(dnp no)
 		(fields_autoplaced yes)
-		(property "Reference" "C708"
+		(property "Reference" "C710"
 			(at 162.56 80.0163 0)
 			(effects
@@
 			(project "ESP_bare_chip_test_board"
 				(path "/45b6f84a-e69b-48be-a49b-bc68872e2c15/01bb46e3-d129-4909-82a1-6bb013dc8f71/9be7d96f-e7c5-43f0-93fa-5964acc52bec"
-					(reference "C708")
+					(reference "C710")
 					(unit 1)
 				)
@@
 		(dnp no)
 		(fields_autoplaced yes)
-		(property "Reference" "C706"
+		(property "Reference" "C708"
 			(at 127 69.8563 0)
 			(effects
@@
 			(project "ESP_bare_chip_test_board"
 				(path "/45b6f84a-e69b-48be-a49b-bc68872e2c15/01bb46e3-d129-4909-82a1-6bb013dc8f71/9be7d96f-e7c5-43f0-93fa-5964acc52bec"
-					(reference "C706")
+					(reference "C708")
 					(unit 1)
 				)
@@
 		(on_board yes)
 		(dnp no)
-		(property "Reference" "C709"
+		(property "Reference" "C701"
 			(at 49.784 147.955 0)
 			(effects
@@
 			(project "ESP_bare_chip_test_board"
 				(path "/45b6f84a-e69b-48be-a49b-bc68872e2c15/01bb46e3-d129-4909-82a1-6bb013dc8f71/9be7d96f-e7c5-43f0-93fa-5964acc52bec"
-					(reference "C709")
+					(reference "C701")
 					(unit 1)
 				)
@@
 		(dnp yes)
 		(fields_autoplaced yes)
-		(property "Reference" "C702"
+		(property "Reference" "C704"
 			(at 93.98 69.8563 0)
 			(effects
@@
 			(project "ESP_bare_chip_test_board"
 				(path "/45b6f84a-e69b-48be-a49b-bc68872e2c15/01bb46e3-d129-4909-82a1-6bb013dc8f71/9be7d96f-e7c5-43f0-93fa-5964acc52bec"
-					(reference "C702")
+					(reference "C704")
 					(unit 1)
 				)
@@
 		(dnp no)
 		(fields_autoplaced yes)
-		(property "Reference" "#PWR0710"
+		(property "Reference" "#PWR0707"
 			(at 139.7 166.37 0)
 			(effects
@@
 			(project "ESP_bare_chip_test_board"
 				(path "/45b6f84a-e69b-48be-a49b-bc68872e2c15/01bb46e3-d129-4909-82a1-6bb013dc8f71/9be7d96f-e7c5-43f0-93fa-5964acc52bec"
-					(reference "#PWR0710")
+					(reference "#PWR0707")
 					(unit 1)
 				)
@@
 		(dnp no)
 		(fields_autoplaced yes)
-		(property "Reference" "C704"
+		(property "Reference" "C706"
 			(at 114.3 69.8563 0)
 			(effects
@@
 			(project "ESP_bare_chip_test_board"
 				(path "/45b6f84a-e69b-48be-a49b-bc68872e2c15/01bb46e3-d129-4909-82a1-6bb013dc8f71/9be7d96f-e7c5-43f0-93fa-5964acc52bec"
-					(reference "C704")
-					(unit 1)
-				)
+					(reference "C706")
+					(unit 1)
+				)
