File: subsheet/step-down-12v-5v.kicad_sch (KiCad schematic)
At the start: 11 parts, among them U1101 TPS563201

Commit message: PCB changes, added useful connectors
Added a whole bunch of things that should make it useful - e.g.
ethernet, an extra flash chip for general storage, piicodev connectors
for I2C.

Also added a GPIB connector footprint; dev-board version worked nicely,
but may as well make this work for that too. Saves bying dev boards : )
Parts:
- renumbered C1101 to C1601, C1102 to C1602, C1103 to C1603, C1106 to C?, C1105 to C?, C1107 to C?, C1104 to C?, L1101 to L1601, R1101 to R1601, R1102 to R1602, U1101 to U1601
Other:
- note added: "Note: Be careful about how close the Boot capacitor and FB resistor are to each other! If the high-frequency switching couples from BOOT to the FB pin, it will mess up the voltage regulation I encountered this while tesing v4.0.0: I touched them with my (dry) fingertip, causing an AC short between BOOT the FB pins on the resistors. The inductor would buzz, and board would stop working after 2 or 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"
Changed lines of the file:
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@@
+		)
+	)
+	(text "Note: Be careful about how close the Boot capacitor and\nFB resistor are to each other! If the high-frequency switching\ncouples from BOOT to the FB pin, it will mess up the voltage regulation\n\nI encountered this while tesing v4.0.0: I touched them\nwith my (dry) fingertip, causing an AC short between BOOT\nthe FB pins on the resistors. The inductor would buzz, \nand board would stop working after 2 or 3 times.\n\nForum post that explains the issue:\nhttps://e2e.ti.com/support/power-management-group/power-management/f/power-management-forum/623443/tps563200-output-spike-when-touched-part-toasted\n\n"
+		(exclude_from_sim no)
+		(at 22.86 187.96 0)
+		(effects
+			(font
+				(size 2.54 2.54)
+			)
+			(justify left)
 		)
 	)
@@
 		(on_board yes)
 		(dnp no)
-		(property "Reference" "C1106"
+		(property "Reference" "C?"
 			(at 202.184 102.235 0)
 			(effects
@@
 		)
 		(instances
+			(project "Nokia-3310-ESP32"
+				(path "/1b0b2d77-639c-42d7-8c01-0ca0be561a47/a8e9a14a-6d9a-4a33-90ba-a3291f378bd4"
+					(reference "C?")
+					(unit 1)
+				)
+			)
 			(project "ESP_bare_chip_test_board"
 				(path "/45b6f84a-e69b-48be-a49b-bc68872e2c15/28425a28-8968-4679-b18b-58814452f93f/f2eaccf6-891f-4f8c-bb6d-39d189e94a7d"
-					(reference "C1106")
+					(reference "C?")
+					(unit 1)
+				)
+			)
+			(project "puzzle-shield-ESP32"
+				(path "/7f264da7-ad23-4f41-956f-57553b2e7107/5a6cdf82-c956-4eb3-893f-6bfd5dd30cf7/642e6ca5-36c0-4ff3-900b-bea7baeb62cc"
+					(reference "C1606")
 					(unit 1)
 				)
@@
 		(dnp no)
 		(fields_autoplaced yes)
-		(property "Reference" "#PWR01101"
+		(property "Reference" "#PWR01601"
 			(at 119.38 123.19 0)
 			(effects
@@
 			(project "ESP_bare_chip_test_board"
 				(path "/45b6f84a-e69b-48be-a49b-bc68872e2c15/28425a28-8968-4679-b18b-58814452f93f/f2eaccf6-891f-4f8c-bb6d-39d189e94a7d"
-					(reference "#PWR01101")
+					(reference "#PWR01601")
+					(unit 1)
+				)
+			)
+			(project "puzzle-shield-ESP32"
+				(path "/7f264da7-ad23-4f41-956f-57553b2e7107/5a6cdf82-c956-4eb3-893f-6bfd5dd30cf7/642e6ca5-36c0-4ff3-900b-bea7baeb62cc"
+					(reference "#PWR01601")
 					(unit 1)
 				)
@@
 		(on_board yes)
 		(dnp no)
-		(property "Reference" "C1101"
+		(property "Reference" "C1601"
 			(at 75.9968 100.4316 0)
 			(effects
@@
 			(project "ESP_bare_chip_test_board"
 				(path "/45b6f84a-e69b-48be-a49b-bc68872e2c15/28425a28-8968-4679-b18b-58814452f93f/f2eaccf6-891f-4f8c-bb6d-39d189e94a7d"
-					(reference "C1101")
+					(reference "C1601")
+					(unit 1)
+				)
+			)
+			(project "puzzle-shield-ESP32"
+				(path "/7f264da7-ad23-4f41-956f-57553b2e7107/5a6cdf82-c956-4eb3-893f-6bfd5dd30cf7/642e6ca5-36c0-4ff3-900b-bea7baeb62cc"
+					(reference "C1601")
 					(unit 1)
 				)
@@
 		(on_board yes)
 		(dnp no)
-		(property "Reference" "C1105"
+		(property "Reference" "C?"
 			(at 186.944 102.235 0)
 			(effects
@@
 		)
 		(instances
+			(project "Nokia-3310-ESP32"
+				(path "/1b0b2d77-639c-42d7-8c01-0ca0be561a47/a8e9a14a-6d9a-4a33-90ba-a3291f378bd4"
+					(reference "C?")
+					(unit 1)
+				)
+			)
 			(project "ESP_bare_chip_test_board"
 				(path "/45b6f84a-e69b-48be-a49b-bc68872e2c15/28425a28-8968-4679-b18b-58814452f93f/f2eaccf6-891f-4f8c-bb6d-39d189e94a7d"
-					(reference "C1105")
+					(reference "C?")
+					(unit 1)
+				)
+			)
+			(project "puzzle-shield-ESP32"
+				(path "/7f264da7-ad23-4f41-956f-57553b2e7107/5a6cdf82-c956-4eb3-893f-6bfd5dd30cf7/642e6ca5-36c0-4ff3-900b-bea7baeb62cc"
+					(reference "C1605")
 					(unit 1)
 				)
@@
 		(on_board yes)
 		(dnp no)
-		(property "Reference" "C1102"
+		(property "Reference" "C1602"
 			(at 91.2368 100.4316 0)
 			(effects
@@
 			(project "ESP_bare_chip_test_board"
 				(path "/45b6f84a-e69b-48be-a49b-bc68872e2c15/28425a28-8968-4679-b18b-58814452f93f/f2eaccf6-891f-4f8c-bb6d-39d189e94a7d"
-					(reference "C1102")
+					(reference "C1602")
+					(unit 1)
+				)
+			)
+			(project "puzzle-shield-ESP32"
+				(path "/7f264da7-ad23-4f41-956f-57553b2e7107/5a6cdf82-c956-4eb3-893f-6bfd5dd30cf7/642e6ca5-36c0-4ff3-900b-bea7baeb62cc"
+					(reference "C1602")
 					(unit 1)
 				)
@@
 		(on_board yes)
 		(dnp no)
-		(property "Reference" "C1107"
+		(property "Reference" "C?"
 			(at 217.424 102.235 0)
 			(effects
@@
 		)
 		(instances
+			(project "Nokia-3310-ESP32"
+				(path "/1b0b2d77-639c-42d7-8c01-0ca0be561a47/a8e9a14a-6d9a-4a33-90ba-a3291f378bd4"
+					(reference "C?")
+					(unit 1)
+				)
+			)
 			(project "ESP_bare_chip_test_board"
 				(path "/45b6f84a-e69b-48be-a49b-bc68872e2c15/28425a28-8968-4679-b18b-58814452f93f/f2eaccf6-891f-4f8c-bb6d-39d189e94a7d"
-					(reference "C1107")
+					(reference "C?")
+					(unit 1)
+				)
+			)
+			(project "puzzle-shield-ESP32"
+				(path "/7f264da7-ad23-4f41-956f-57553b2e7107/5a6cdf82-c956-4eb3-893f-6bfd5dd30cf7/642e6ca5-36c0-4ff3-900b-bea7baeb62cc"
+					(reference "C1607")
 					(unit 1)
 				)
@@
 		(dnp no)
 		(fields_autoplaced yes)
-		(property "Reference" "C1103"
+		(property "Reference" "C1603"
 			(at 142.0368 95.3516 0)
 			(effects
@@
 			(project "ESP_bare_chip_test_board"
 				(path "/45b6f84a-e69b-48be-a49b-bc68872e2c15/28425a28-8968-4679-b18b-58814452f93f/f2eaccf6-891f-4f8c-bb6d-39d189e94a7d"
-					(reference "C1103")
+					(reference "C1603")
+					(unit 1)
+				)
+			)
+			(project "puzzle-shield-ESP32"
+				(path "/7f264da7-ad23-4f41-956f-57553b2e7107/5a6cdf82-c956-4eb3-893f-6bfd5dd30cf7/642e6ca5-36c0-4ff3-900b-bea7baeb62cc"
+					(reference "C1603")
 					(unit 1)
 				)
@@
 		(on_board yes)
 		(dnp no)
-		(property "Reference" "R1101"
+		(property "Reference" "R1601"
 			(at 154.1272 97.8916 0)
 			(effects
@@
 			(project "ESP_bare_chip_test_board"
 				(path "/45b6f84a-e69b-48be-a49b-bc68872e2c15/28425a28-8968-4679-b18b-58814452f93f/f2eaccf6-891f-4f8c-bb6d-39d189e94a7d"
-					(reference "R1101")
+					(reference "R1601")
+					(unit 1)
+				)
+			)
+			(project "puzzle-shield-ESP32"
+				(path "/7f264da7-ad23-4f41-956f-57553b2e7107/5a6cdf82-c956-4eb3-893f-6bfd5dd30cf7/642e6ca5-36c0-4ff3-900b-bea7baeb62cc"
+					(reference "R1601")
 					(unit 1)
 				)
@@
 		(dnp no)
 		(fields_autoplaced yes)
-		(property "Reference" "L1101"
+		(property "Reference" "L1601"
 			(at 146.05 86.36 90)
 			(effects
@@
 			(project "ESP_bare_chip_test_board"
 				(path "/45b6f84a-e69b-48be-a49b-bc68872e2c15/28425a28-8968-4679-b18b-58814452f93f/f2eaccf6-891f-4f8c-bb6d-39d189e94a7d"
-					(reference "L1101")
+					(reference "L1601")
+					(unit 1)
+				)
+			)
+			(project "puzzle-shield-ESP32"
+				(path "/7f264da7-ad23-4f41-956f-57553b2e7107/5a6cdf82-c956-4eb3-893f-6bfd5dd30cf7/642e6ca5-36c0-4ff3-900b-bea7baeb62cc"
+					(reference "L1601")
 					(unit 1)
 				)
@@
 		(on_board yes)
 		(dnp no)
-		(property "Reference" "R1102"
+		(property "Reference" "R1602"
 			(at 154.1272 108.0516 0)
 			(effects
@@
 			(project "ESP_bare_chip_test_board"
 				(path "/45b6f84a-e69b-48be-a49b-bc68872e2c15/28425a28-8968-4679-b18b-58814452f93f/f2eaccf6-891f-4f8c-bb6d-39d189e94a7d"
-					(reference "R1102")
+					(reference "R1602")
+					(unit 1)
+				)
+			)
+			(project "puzzle-shield-ESP32"
+				(path "/7f264da7-ad23-4f41-956f-57553b2e7107/5a6cdf82-c956-4eb3-893f-6bfd5dd30cf7/642e6ca5-36c0-4ff3-900b-bea7baeb62cc"
+					(reference "R1602")
 					(unit 1)
 				)
@@
 		(on_board yes)
 		(dnp no)
-		(property "Reference" "C1104"
+		(property "Reference" "C?"
 			(at 171.704 102.235 0)
 			(effects
@@
 		)
 		(instances
+			(project "Nokia-3310-ESP32"
+				(path "/1b0b2d77-639c-42d7-8c01-0ca0be561a47/a8e9a14a-6d9a-4a33-90ba-a3291f378bd4"
+					(reference "C?")
+					(unit 1)
+				)
+			)
 			(project "ESP_bare_chip_test_board"
 				(path "/45b6f84a-e69b-48be-a49b-bc68872e2c15/28425a28-8968-4679-b18b-58814452f93f/f2eaccf6-891f-4f8c-bb6d-39d189e94a7d"
-					(reference "C1104")
+					(reference "C?")
+					(unit 1)
+				)
+			)
+			(project "puzzle-shield-ESP32"
+				(path "/7f264da7-ad23-4f41-956f-57553b2e7107/5a6cdf82-c956-4eb3-893f-6bfd5dd30cf7/642e6ca5-36c0-4ff3-900b-bea7baeb62cc"
+					(reference "C1604")
 					(unit 1)
 				)
@@
 		(dnp no)
 		(fields_autoplaced yes)
-		(property "Reference" "U1101"
+		(property "Reference" "U1601"
 			(at 119.38 83.82 0)
 			(effects
@@
 			(project "ESP_bare_chip_test_board"
 				(path "/45b6f84a-e69b-48be-a49b-bc68872e2c15/28425a28-8968-4679-b18b-58814452f93f/f2eaccf6-891f-4f8c-bb6d-39d189e94a7d"
-					(reference "U1101")
-					(unit 1)
-				)
+					(reference "U1601")
+					(unit 1)
+				)
+			)
+			(project "puzzle-shield-ESP32"
+				(path "/7f264da7-ad23-4f41-956f-57553b2e7107/5a6cdf82-c956-4eb3-893f-6bfd5dd30cf7/642e6ca5-36c0-4ff3-900b-bea7baeb62cc"
+					(reference "U1601")
+					(unit 1)
+				)

Commit message: Uknown changes?File formats?
Parts:
- renumbered C1601 to C1101, C1602 to C1102, C1603 to C1103, L1601 to L1101, R1601 to R1101, R1602 to R1102, U1601 to U1101
Changed lines of the file:
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@@
 			(project "ESP_bare_chip_test_board"
 				(path "/45b6f84a-e69b-48be-a49b-bc68872e2c15/28425a28-8968-4679-b18b-58814452f93f/f2eaccf6-891f-4f8c-bb6d-39d189e94a7d"
-					(reference "C?")
+					(reference "C1106")
 					(unit 1)
 				)
@@
 		(dnp no)
 		(fields_autoplaced yes)
-		(property "Reference" "#PWR01601"
+		(property "Reference" "#PWR01101"
 			(at 119.38 123.19 0)
 			(effects
@@
 			(project "ESP_bare_chip_test_board"
 				(path "/45b6f84a-e69b-48be-a49b-bc68872e2c15/28425a28-8968-4679-b18b-58814452f93f/f2eaccf6-891f-4f8c-bb6d-39d189e94a7d"
-					(reference "#PWR01601")
+					(reference "#PWR01101")
 					(unit 1)
 				)
@@
 		(on_board yes)
 		(dnp no)
-		(property "Reference" "C1601"
+		(property "Reference" "C1101"
 			(at 75.9968 100.4316 0)
 			(effects
@@
 			(project "ESP_bare_chip_test_board"
 				(path "/45b6f84a-e69b-48be-a49b-bc68872e2c15/28425a28-8968-4679-b18b-58814452f93f/f2eaccf6-891f-4f8c-bb6d-39d189e94a7d"
-					(reference "C1601")
+					(reference "C1101")
 					(unit 1)
 				)
@@
 			(project "ESP_bare_chip_test_board"
 				(path "/45b6f84a-e69b-48be-a49b-bc68872e2c15/28425a28-8968-4679-b18b-58814452f93f/f2eaccf6-891f-4f8c-bb6d-39d189e94a7d"
-					(reference "C?")
+					(reference "C1105")
 					(unit 1)
 				)
@@
 		(on_board yes)
 		(dnp no)
-		(property "Reference" "C1602"
+		(property "Reference" "C1102"
 			(at 91.2368 100.4316 0)
 			(effects
@@
 			(project "ESP_bare_chip_test_board"
 				(path "/45b6f84a-e69b-48be-a49b-bc68872e2c15/28425a28-8968-4679-b18b-58814452f93f/f2eaccf6-891f-4f8c-bb6d-39d189e94a7d"
-					(reference "C1602")
+					(reference "C1102")
 					(unit 1)
 				)
@@
 			(project "ESP_bare_chip_test_board"
 				(path "/45b6f84a-e69b-48be-a49b-bc68872e2c15/28425a28-8968-4679-b18b-58814452f93f/f2eaccf6-891f-4f8c-bb6d-39d189e94a7d"
-					(reference "C?")
+					(reference "C1107")
 					(unit 1)
 				)
@@
 		(dnp no)
 		(fields_autoplaced yes)
-		(property "Reference" "C1603"
+		(property "Reference" "C1103"
 			(at 142.0368 95.3516 0)
 			(effects
@@
 			(project "ESP_bare_chip_test_board"
 				(path "/45b6f84a-e69b-48be-a49b-bc68872e2c15/28425a28-8968-4679-b18b-58814452f93f/f2eaccf6-891f-4f8c-bb6d-39d189e94a7d"
-					(reference "C1603")
+					(reference "C1103")
 					(unit 1)
 				)
@@
 		(on_board yes)
 		(dnp no)
-		(property "Reference" "R1601"
+		(property "Reference" "R1101"
 			(at 154.1272 97.8916 0)
 			(effects
@@
 			(project "ESP_bare_chip_test_board"
 				(path "/45b6f84a-e69b-48be-a49b-bc68872e2c15/28425a28-8968-4679-b18b-58814452f93f/f2eaccf6-891f-4f8c-bb6d-39d189e94a7d"
-					(reference "R1601")
+					(reference "R1101")
 					(unit 1)
 				)
@@
 		(dnp no)
 		(fields_autoplaced yes)
-		(property "Reference" "L1601"
+		(property "Reference" "L1101"
 			(at 146.05 86.36 90)
 			(effects
@@
 			(project "ESP_bare_chip_test_board"
 				(path "/45b6f84a-e69b-48be-a49b-bc68872e2c15/28425a28-8968-4679-b18b-58814452f93f/f2eaccf6-891f-4f8c-bb6d-39d189e94a7d"
-					(reference "L1601")
+					(reference "L1101")
 					(unit 1)
 				)
@@
 		(on_board yes)
 		(dnp no)
-		(property "Reference" "R1602"
+		(property "Reference" "R1102"
 			(at 154.1272 108.0516 0)
 			(effects
@@
 			(project "ESP_bare_chip_test_board"
 				(path "/45b6f84a-e69b-48be-a49b-bc68872e2c15/28425a28-8968-4679-b18b-58814452f93f/f2eaccf6-891f-4f8c-bb6d-39d189e94a7d"
-					(reference "R1602")
+					(reference "R1102")
 					(unit 1)
 				)
@@
 			(project "ESP_bare_chip_test_board"
 				(path "/45b6f84a-e69b-48be-a49b-bc68872e2c15/28425a28-8968-4679-b18b-58814452f93f/f2eaccf6-891f-4f8c-bb6d-39d189e94a7d"
-					(reference "C?")
+					(reference "C1104")
 					(unit 1)
 				)
@@
 		(dnp no)
 		(fields_autoplaced yes)
-		(property "Reference" "U1601"
+		(property "Reference" "U1101"
 			(at 119.38 83.82 0)
 			(effects
@@
 			(project "ESP_bare_chip_test_board"
 				(path "/45b6f84a-e69b-48be-a49b-bc68872e2c15/28425a28-8968-4679-b18b-58814452f93f/f2eaccf6-891f-4f8c-bb6d-39d189e94a7d"
-					(reference "U1601")
-					(unit 1)
-				)
+					(reference "U1101")
+					(unit 1)
+				)
