File: subsheet/ESP32-S3-core.kicad_sch (KiCad schematic)
At the start: 22 parts, among them Q601 40MHz, U7 W25Q128JVS, U8 ESP32-S3

Commit message: Copy in component arrangement from SDMMC test design
Already had an efficient arrangement for the SPI flash chip, Clock
crystal, and Antenna.
Parts:
- renumbered C703 to C303, C704 to C304, C705 to C305, C706 to C306, C707 to C307, C708 to C308, C709 to C309, C710 to C310, C711 to C311, C712 to C312, L701 to L301, R701 to R301, R702 to R302, R703 to R303, R704 to R304, R705 to R305, R706 to R306, U7 to U301, U8 to U302

Commit message: Picked part numbers and placed most remaining MCU support components
Parts:
- C303: value 10uF -> 10uF/10V; footprint (none) -> Capacitor_SMD:C_0603_1608Metric; LCSC (none) -> C19702
- C304, C306, C309: footprint (none) -> Capacitor_SMD:C_0402_1005Metric
- L301: footprint (none) -> Inductor_SMD:L_0402_1005Metric; LCSC (none) -> C43365
- R301: value TBD, 24nH to start -> 24nH; Comment (none) -> TBD; LCSC (none) -> C330863
Other:
- note added: "Value of R301 TBD Can be inductor or resistor Reccomend 24nH to start"

Commit message: Add order codes for all components
Parts:
- C304, C305, C307: LCSC (none) -> C52923
- C306, C309, C310, C311, C312: LCSC (none) -> C307331
- C308: LCSC (none) -> C15195
- R302, R303, R304, R305, R306: LCSC (none) -> C203078
- U302: LCSC (none) -> C2913192

Commit message: Switch to ESP32-S3R8 (8Mb PSRAM)
Switch to the ESP32-S3 chip that has integrated PSRAM, so I can test it
Disadvantage is it means IO26 cannot be used, and is more expensive.
Still uses external flash chip.
Parts:
- U302: value ESP32-S3 -> ESP32-S3R8; LCSC C2913192 -> C2913194
Changed lines of the file:
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@@
 			)
 		)
-		(property "Value" "ESP32-S3"
+		(property "Value" "ESP32-S3R8"
 			(at 146.9741 160.02 0)
 			(effects
@@
 			)
 		)
-		(property "LCSC" "C2913192"
+		(property "LCSC" "C2913194"
 			(at 144.78 116.84 0)
 			(effects

Commit message: Add JLCPCB corrections for new components
Parts:
- Q601: JLCPCB_CORRECTION (none) -> 0;0;0
- U301: JLCPCB_CORRECTION (none) -> 0;0;270
Changed lines of the file:
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@@
+			)
+		)
+		(property "JLCPCB_CORRECTION" "0;0;0"
+			(at 54.61 119.38 0)
+			(effects
+				(font
+					(size 1.27 1.27)
+				)
+				(hide yes)
 			)
 		)
@@
 			(at 116.84 177.8 0)
 			(effects
+				(font
+					(size 1.27 1.27)
+				)
+				(hide yes)
+			)
+		)
+		(property "JLCPCB_CORRECTION" "0;0;270"
+			(at 116.84 177.8 0)
+			(effects

Commit message: Silkscreen work. Edit tittle block/version number
Other:
- company: (none) -> (c) Vincent Dalstra
- title: (none) -> Untitled 4-layer JLCPCB
Changed lines of the file:
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@@
 	(generator_version "8.0")
 	(paper "A4")
+	(title_block
+		(title "Untitled 4-layer JLCPCB")
+		(date "2024-06-14")
+		(rev "1.0.0")
+		(company "(c) Vincent Dalstra")
+	)
 	(junction
 		(at 162.56 55.88)
