File: subsheet/ESP32-S3.kicad_sch (KiCad schematic)
At the start: 10 parts, among them J201 Conn_01x06, SW201 SW_Push, SW202 SW_Push, U201 ESP32-S3-MINI-1

Commit message: Add JLCPCB corrections for new components
Parts:
- D201: JLCPCB_CORRECTION (none) -> 0;0;0; LCSC C72043 -> C779453
- J201: JLCPCB_IGNORE (none) -> 1
Changed lines of the file:
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@@
 			)
 		)
-		(property "LCSC" "C72043"
+		(property "LCSC" "C779453"
 			(at 243.84 22.86 0)
 			(effects
@@
 		)
 		(property "I2C address" ""
+			(at 243.84 22.86 0)
+			(effects
+				(font
+					(size 1.27 1.27)
+				)
+				(hide yes)
+			)
+		)
+		(property "JLCPCB_CORRECTION" "0;0;0"
 			(at 243.84 22.86 0)
 			(effects
@@
 			(at 25.4 82.55 0)
 			(effects
+				(font
+					(size 1.27 1.27)
+				)
+				(hide yes)
+			)
+		)
+		(property "JLCPCB_IGNORE" "1"
+			(at 25.4 82.55 0)
+			(effects

Commit message: Silkscreen work. Edit tittle block/version number
Other:
- company: (c) Escape This -> (c) Vincent Dalstra
- title: Environment Controller ESP32-S3-4M -> Untitled 4-layer JLCPCB
Changed lines of the file:
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@@
 	(paper "A4")
 	(title_block
-		(title "Environment Controller ESP32-S3-4M")
-		(date "2023-08-16")
-		(rev "1.1.0")
-		(company "(c) Escape This")
+		(title "Untitled 4-layer JLCPCB")
+		(date "2024-06-14")
+		(rev "1.0.0")
+		(company "(c) Vincent Dalstra")
 		(comment 1 "Drawn by: VGD")
 		(comment 2 "Check by:")

Commit message: Move all subsheets into 'main' subsheet, below root
Keeping all the subsheets in a dedicated 'subsheet' folder makes things
much, much neater. However, specifying filepaths for subsheets has an
interesting problem; they use paths RELATIVE TO THE PARENT SHEET.

The consequence of is that if a subsheet is part of the root sheet, it
needs to be prefixed with 'subsheet/', but NOT if it's further down.
This inconsistency can be resolved by having a single 'main' sheet at
the top that doesn't move.

It's also useful to have a top-level space to put down changelogs,
descriptions etc.
Parts:
- renumbered C201 to C301, C202 to C302, C203 to C303, D201 to D301, J201 to J301, R201 to R301, R202 to R302, SW201 to SW301, SW202 to SW302, U201 to U301
