File: subsheet/Power.kicad_sch (KiCad schematic)
At the start: 12 parts, among them J501 Barrel_Jack, J502 PWR_IN, J503 ALTERNATE

Commit message: Silkscreen work. Edit tittle block/version number
Other:
- company: (none) -> (c) Vincent Dalstra
- title: (none) -> Untitled 4-layer JLCPCB
Changed lines of the file:
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@@
 	(generator_version "8.0")
 	(paper "A4")
+	(title_block
+		(title "Untitled 4-layer JLCPCB")
+		(date "2024-06-14")
+		(rev "1.0.0")
+		(company "(c) Vincent Dalstra")
+	)
 	(junction
 		(at 60.96 127)

Commit message: Move all subsheets into 'main' subsheet, below root
Keeping all the subsheets in a dedicated 'subsheet' folder makes things
much, much neater. However, specifying filepaths for subsheets has an
interesting problem; they use paths RELATIVE TO THE PARENT SHEET.

The consequence of is that if a subsheet is part of the root sheet, it
needs to be prefixed with 'subsheet/', but NOT if it's further down.
This inconsistency can be resolved by having a single 'main' sheet at
the top that doesn't move.

It's also useful to have a top-level space to put down changelogs,
descriptions etc.
Parts:
- renumbered C501 to C701, D501 to D701, D502 to D702, D503 to D703, D504 to D704, D505 to D705, D509 to D706, D507 to D707, J501 to J701, J502 to J702, J503 to J703, R506 to R701

Commit message: Update file format to KiCAD 9.0
Changed lines of the file:
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@@
 (kicad_sch
-	(version 20231120)
+	(version 20250114)
 	(generator "eeschema")
-	(generator_version "8.0")
+	(generator_version "9.0")
 	(paper "A4")
 	(title_block
@@
 		(company "(c) Vincent Dalstra")
 	)
+	(text "For a USB-C Sink, C_{VBUS} <= 10uF\n- Another 90uF is allowed after the\n	over-voltage protection switch.\n"
+		(exclude_from_sim no)
+		(at 15.24 38.1 0)
+		(effects
+			(font
+				(size 1.27 1.27)
+			)
+			(justify left bottom)
+		)
+	)
+	(text "Terminal Plug: C560212"
+		(exclude_from_sim no)
+		(at 15.24 134.62 90)
+		(effects
+			(font
+				(size 1.27 1.27)
+			)
+			(justify left bottom)
+		)
+	)
+	(text "One regulator provides powe to the ESP32 and the\nEthernet module. It also supplies the Piicodev\nconnectors (via a load-switch with 1.1A limit).\n\nThe other regulator supplies 3v3 to the IO connectors,\nso that overload/noise will not interfere with the ESP32.\nIt also makes routing simpler."
+		(exclude_from_sim no)
+		(at 226.06 114.3 0)
+		(effects
+			(font
+				(size 1.27 1.27)
+			)
+			(justify left bottom)
+		)
+	)
+	(text "TPS2552\n- 5V 1.5A load switch (7.0V absMAX)\n- overcurrent protection (programmable)\n- short circuit protection \n- Reverse-voltage protection"
+		(exclude_from_sim no)
+		(at 88.9 -2.54 0)
+		(effects
+			(font
+				(size 1.27 1.27)
+			)
+			(justify left bottom)
+		)
+	)
+	(text "Inefficient, but simple"
+		(exclude_from_sim no)
+		(at 101.6 83.82 0)
+		(effects
+			(font
+				(size 1.27 1.27)
+			)
+		)
+	)
+	(text "Todo: add 28V OVP load-switch AW32905FCR (C401023)\nto protect the TPS2552 from voltages greater than 6.5V\n- Also provides ESD/surge protection (up to 120V)\n- OTG functionality allows 0V drop in reverse (like a P-mosfet)\n	- First the internal body diode conducts to 2.5V\n	- Then the mosfet is driven high to remove the voltage drop\n"
+		(exclude_from_sim no)
+		(at -2.54 7.62 0)
+		(effects
+			(font
+				(size 1.27 1.27)
+			)
+			(justify left bottom)
+		)
+	)
+	(text "V_{IN} 2-16V\n(20V abs. max.)"
+		(exclude_from_sim no)
+		(at 127 127 0)
+		(effects
+			(font
+				(size 1.27 1.27)
+			)
+			(justify left top)
+		)
+	)
+	(text "Override names"
+		(exclude_from_sim no)
+		(at 10.16 213.36 0)
+		(effects
+			(font
+				(size 1.27 1.27)
+			)
+			(justify left bottom)
+		)
+	)
+	(text "Todo: replace with SS54 or SS34\n(Lower reverse-breakdown, but gain\nlower forward-voltage in return)"
+		(exclude_from_sim no)
+		(at 81.28 154.94 0)
+		(effects
+			(font
+				(size 1.27 1.27)
+			)
+		)
+	)
+	(text "Resistors target for\napprox. 0.1mA"
+		(exclude_from_sim no)
+		(at 129.54 181.61 0)
+		(effects
+			(font
+				(size 1.27 1.27)
+			)
+			(justify left bottom)
+		)
+	)
+	(text "PGOOD is\nopen-drain"
+		(exclude_from_sim no)
+		(at 160.02 142.24 0)
+		(effects
+			(font
+				(size 1.27 1.27)
+			)
+			(justify left)
+		)
+	)
 	(junction
 		(at 60.96 127)
@@
 			(width 0)
 			(type default)
-		)
-	)
-	(text "For a USB-C Sink, C_{VBUS} <= 10uF\n- Another 90uF is allowed after the\n	over-voltage protection switch.\n"
-		(exclude_from_sim no)
-		(at 15.24 38.1 0)
-		(effects
-			(font
-				(size 1.27 1.27)
-			)
-			(justify left bottom)
-		)
-	)
-	(text "Terminal Plug: C560212"
-		(exclude_from_sim no)
-		(at 15.24 134.62 90)
-		(effects
-			(font
-				(size 1.27 1.27)
-			)
-			(justify left bottom)
-		)
-	)
-	(text "One regulator provides powe to the ESP32 and the\nEthernet module. It also supplies the Piicodev\nconnectors (via a load-switch with 1.1A limit).\n\nThe other regulator supplies 3v3 to the IO connectors,\nso that overload/noise will not interfere with the ESP32.\nIt also makes routing simpler."
-		(exclude_from_sim no)
-		(at 226.06 114.3 0)
-		(effects
-			(font
-				(size 1.27 1.27)
-			)
-			(justify left bottom)
-		)
-	)
-	(text "TPS2552\n- 5V 1.5A load switch (7.0V absMAX)\n- overcurrent protection (programmable)\n- short circuit protection \n- Reverse-voltage protection"
-		(exclude_from_sim no)
-		(at 88.9 -2.54 0)
-		(effects
-			(font
-				(size 1.27 1.27)
-			)
-			(justify left bottom)
-		)
-	)
-	(text "Inefficient, but simple"
-		(exclude_from_sim no)
-		(at 101.6 83.82 0)
-		(effects
-			(font
-				(size 1.27 1.27)
-			)
-		)
-	)
-	(text "Todo: add 28V OVP load-switch AW32905FCR (C401023)\nto protect the TPS2552 from voltages greater than 6.5V\n- Also provides ESD/surge protection (up to 120V)\n- OTG functionality allows 0V drop in reverse (like a P-mosfet)\n	- First the internal body diode conducts to 2.5V\n	- Then the mosfet is driven high to remove the voltage drop\n"
-		(exclude_from_sim no)
-		(at -2.54 7.62 0)
-		(effects
-			(font
-				(size 1.27 1.27)
-			)
-			(justify left bottom)
-		)
-	)
-	(text "V_{IN} 2-16V\n(20V abs. max.)"
-		(exclude_from_sim no)
-		(at 127 127 0)
-		(effects
-			(font
-				(size 1.27 1.27)
-			)
-			(justify left top)
-		)
-	)
-	(text "Override names"
-		(exclude_from_sim no)
-		(at 10.16 213.36 0)
-		(effects
-			(font
-				(size 1.27 1.27)
-			)
-			(justify left bottom)
-		)
-	)
-	(text "Todo: replace with SS54 or SS34\n(Lower reverse-breakdown, but gain\nlower forward-voltage in return)"
-		(exclude_from_sim no)
-		(at 81.28 154.94 0)
-		(effects
-			(font
-				(size 1.27 1.27)
-			)
-		)
-	)
-	(text "Resistors target for\napprox. 0.1mA"
-		(exclude_from_sim no)
-		(at 129.54 181.61 0)
-		(effects
-			(font
-				(size 1.27 1.27)
-			)
-			(justify left bottom)
-		)
-	)
-	(text "PGOOD is\nopen-drain"
-		(exclude_from_sim no)
-		(at 160.02 142.24 0)
-		(effects
-			(font
-				(size 1.27 1.27)
-			)
-			(justify left)
 		)
 	)
@@
 		(at 144.78 129.54)
 		(size 12.7 15.24)
+		(exclude_from_sim no)
+		(in_bom yes)
+		(on_board yes)
+		(dnp no)
 		(fields_autoplaced yes)
 		(stroke
@@
 		(at 233.68 144.78)
 		(size 15.24 10.16)
+		(exclude_from_sim no)
+		(in_bom yes)
+		(on_board yes)
+		(dnp no)
 		(fields_autoplaced yes)
 		(stroke
