File: subsheet/buck-boost-5v.kicad_sch (KiCad schematic)
At the start: 13 parts, among them U1002 TPS63070

Commit message: Move all subsheets into 'main' subsheet, below root
Keeping all the subsheets in a dedicated 'subsheet' folder makes things
much, much neater. However, specifying filepaths for subsheets has an
interesting problem; they use paths RELATIVE TO THE PARENT SHEET.

The consequence of is that if a subsheet is part of the root sheet, it
needs to be prefixed with 'subsheet/', but NOT if it's further down.
This inconsistency can be resolved by having a single 'main' sheet at
the top that doesn't move.

It's also useful to have a top-level space to put down changelogs,
descriptions etc.
Parts:
- renumbered C1010 to C801, C1011 to C802, C1012 to C803, C1004 to C804, C1005 to C805, C1006 to C806, C1007 to C807, L1003 to L801, NT901 to NT801, R1003 to R801, R1004 to R802, R1005 to R803, U1002 to U801
Changed lines of the file:
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@@
 	(label "EN_{reg}"
 		(at 99.06 101.6 180)
-		(fields_autoplaced yes)
 		(effects
 			(font
@@
 	(label "MODE"
 		(at 99.06 106.68 180)
-		(fields_autoplaced yes)
 		(effects
 			(font
@@
 	(label "SGND"
 		(at 96.52 157.48 180)
-		(fields_autoplaced yes)
 		(effects
 			(font
@@
 	(label "L1"
 		(at 99.06 86.36 180)
-		(fields_autoplaced yes)
 		(effects
 			(font
@@
 	(label "SGND"
 		(at 111.76 119.38 180)
-		(fields_autoplaced yes)
 		(effects
 			(font
@@
 	(label "V_{AUX}"
 		(at 93.98 111.76 0)
-		(fields_autoplaced yes)
 		(effects
 			(font
@@
 	(label "FB"
 		(at 137.16 101.6 0)
-		(fields_autoplaced yes)
 		(effects
 			(font
@@
 	(label "L2"
 		(at 124.46 86.36 0)
-		(fields_autoplaced yes)
 		(effects
 			(font
@@
 		(shape output)
 		(at 251.46 91.44 0)
-		(fields_autoplaced yes)
 		(effects
 			(font
@@
 		(shape input)
 		(at 22.86 91.44 180)
-		(fields_autoplaced yes)
 		(effects
 			(font
@@
 		(shape output)
 		(at 162.56 66.04 0)
-		(fields_autoplaced yes)
 		(effects
 			(font
@@
 		(on_board yes)
 		(dnp no)
-		(property "Reference" "C1011"
+		(property "Reference" "C802"
 			(at 75.9968 100.4316 0)
 			(effects
@@
 		(instances
 			(project "ESP_bare_chip_test_board"
-				(path "/45b6f84a-e69b-48be-a49b-bc68872e2c15/28425a28-8968-4679-b18b-58814452f93f/a569503a-4f7e-494d-9487-0f55aaa1ce0a"
-					(reference "C1011")
+				(path "/45b6f84a-e69b-48be-a49b-bc68872e2c15/f48098a1-cacc-4192-b650-2a34a2ba76dc/1ca534e3-2263-4539-8aa0-ff724a69b5d8/a569503a-4f7e-494d-9487-0f55aaa1ce0a"
+					(reference "C802")
 					(unit 1)
 				)
@@
 		(dnp no)
 		(fields_autoplaced yes)
-		(property "Reference" "R1004"
+		(property "Reference" "R802"
 			(at 134.62 95.25 0)
 			(effects
@@
 		(instances
 			(project "ESP_bare_chip_test_board"
-				(path "/45b6f84a-e69b-48be-a49b-bc68872e2c15/28425a28-8968-4679-b18b-58814452f93f/a569503a-4f7e-494d-9487-0f55aaa1ce0a"
-					(reference "R1004")
+				(path "/45b6f84a-e69b-48be-a49b-bc68872e2c15/f48098a1-cacc-4192-b650-2a34a2ba76dc/1ca534e3-2263-4539-8aa0-ff724a69b5d8/a569503a-4f7e-494d-9487-0f55aaa1ce0a"
+					(reference "R802")
 					(unit 1)
 				)
@@
 		(on_board yes)
 		(dnp no)
-		(property "Reference" "C1004"
+		(property "Reference" "C804"
 			(at 153.924 104.775 0)
 			(effects
@@
 		(instances
 			(project "ESP_bare_chip_test_board"
-				(path "/45b6f84a-e69b-48be-a49b-bc68872e2c15/28425a28-8968-4679-b18b-58814452f93f/a569503a-4f7e-494d-9487-0f55aaa1ce0a"
-					(reference "C1004")
+				(path "/45b6f84a-e69b-48be-a49b-bc68872e2c15/f48098a1-cacc-4192-b650-2a34a2ba76dc/1ca534e3-2263-4539-8aa0-ff724a69b5d8/a569503a-4f7e-494d-9487-0f55aaa1ce0a"
+					(reference "C804")
 					(unit 1)
 				)
@@
 		(dnp no)
 		(fields_autoplaced yes)
-		(property "Reference" "R1005"
+		(property "Reference" "R803"
 			(at 134.62 105.41 0)
 			(effects
@@
 		(instances
 			(project "ESP_bare_chip_test_board"
-				(path "/45b6f84a-e69b-48be-a49b-bc68872e2c15/28425a28-8968-4679-b18b-58814452f93f/a569503a-4f7e-494d-9487-0f55aaa1ce0a"
-					(reference "R1005")
+				(path "/45b6f84a-e69b-48be-a49b-bc68872e2c15/f48098a1-cacc-4192-b650-2a34a2ba76dc/1ca534e3-2263-4539-8aa0-ff724a69b5d8/a569503a-4f7e-494d-9487-0f55aaa1ce0a"
+					(reference "R803")
 					(unit 1)
 				)
@@
 		(dnp no)
 		(fields_autoplaced yes)
-		(property "Reference" "NT901"
+		(property "Reference" "NT801"
 			(at 99.06 152.4 0)
 			(effects
@@
 		(instances
 			(project "ESP_bare_chip_test_board"
-				(path "/45b6f84a-e69b-48be-a49b-bc68872e2c15/28425a28-8968-4679-b18b-58814452f93f/a569503a-4f7e-494d-9487-0f55aaa1ce0a"
-					(reference "NT901")
+				(path "/45b6f84a-e69b-48be-a49b-bc68872e2c15/f48098a1-cacc-4192-b650-2a34a2ba76dc/1ca534e3-2263-4539-8aa0-ff724a69b5d8/a569503a-4f7e-494d-9487-0f55aaa1ce0a"
+					(reference "NT801")
 					(unit 1)
 				)
@@
 		(on_board yes)
 		(dnp no)
-		(property "Reference" "C1010"
+		(property "Reference" "C801"
 			(at 60.7568 100.4316 0)
 			(effects
@@
 		(instances
 			(project "ESP_bare_chip_test_board"
-				(path "/45b6f84a-e69b-48be-a49b-bc68872e2c15/28425a28-8968-4679-b18b-58814452f93f/a569503a-4f7e-494d-9487-0f55aaa1ce0a"
-					(reference "C1010")
+				(path "/45b6f84a-e69b-48be-a49b-bc68872e2c15/f48098a1-cacc-4192-b650-2a34a2ba76dc/1ca534e3-2263-4539-8aa0-ff724a69b5d8/a569503a-4f7e-494d-9487-0f55aaa1ce0a"
+					(reference "C801")
 					(unit 1)
 				)
@@
 		(dnp no)
 		(fields_autoplaced yes)
-		(property "Reference" "C1012"
+		(property "Reference" "C803"
 			(at 96.3168 118.2116 0)
 			(effects
@@
 		(instances
 			(project "ESP_bare_chip_test_board"
-				(path "/45b6f84a-e69b-48be-a49b-bc68872e2c15/28425a28-8968-4679-b18b-58814452f93f/a569503a-4f7e-494d-9487-0f55aaa1ce0a"
-					(reference "C1012")
+				(path "/45b6f84a-e69b-48be-a49b-bc68872e2c15/f48098a1-cacc-4192-b650-2a34a2ba76dc/1ca534e3-2263-4539-8aa0-ff724a69b5d8/a569503a-4f7e-494d-9487-0f55aaa1ce0a"
+					(reference "C803")
 					(unit 1)
 				)
@@
 		(dnp no)
 		(fields_autoplaced yes)
-		(property "Reference" "U1002"
+		(property "Reference" "U801"
 			(at 111.76 78.74 0)
 			(effects
@@
 		(instances
 			(project "ESP_bare_chip_test_board"
-				(path "/45b6f84a-e69b-48be-a49b-bc68872e2c15/28425a28-8968-4679-b18b-58814452f93f/a569503a-4f7e-494d-9487-0f55aaa1ce0a"
-					(reference "U1002")
+				(path "/45b6f84a-e69b-48be-a49b-bc68872e2c15/f48098a1-cacc-4192-b650-2a34a2ba76dc/1ca534e3-2263-4539-8aa0-ff724a69b5d8/a569503a-4f7e-494d-9487-0f55aaa1ce0a"
+					(reference "U801")
 					(unit 1)
 				)
@@
 		(dnp no)
 		(fields_autoplaced yes)
-		(property "Reference" "R1003"
+		(property "Reference" "R801"
 			(at 88.9 95.25 0)
 			(effects
@@
 		(instances
 			(project "ESP_bare_chip_test_board"
-				(path "/45b6f84a-e69b-48be-a49b-bc68872e2c15/28425a28-8968-4679-b18b-58814452f93f/a569503a-4f7e-494d-9487-0f55aaa1ce0a"
-					(reference "R1003")
+				(path "/45b6f84a-e69b-48be-a49b-bc68872e2c15/f48098a1-cacc-4192-b650-2a34a2ba76dc/1ca534e3-2263-4539-8aa0-ff724a69b5d8/a569503a-4f7e-494d-9487-0f55aaa1ce0a"
+					(reference "R801")
 					(unit 1)
 				)
@@
 		(dnp no)
 		(fields_autoplaced yes)
-		(property "Reference" "L1003"
+		(property "Reference" "L801"
 			(at 110.49 66.04 90)
 			(effects
@@
 		(instances
 			(project "ESP_bare_chip_test_board"
-				(path "/45b6f84a-e69b-48be-a49b-bc68872e2c15/28425a28-8968-4679-b18b-58814452f93f/a569503a-4f7e-494d-9487-0f55aaa1ce0a"
-					(reference "L1003")
+				(path "/45b6f84a-e69b-48be-a49b-bc68872e2c15/f48098a1-cacc-4192-b650-2a34a2ba76dc/1ca534e3-2263-4539-8aa0-ff724a69b5d8/a569503a-4f7e-494d-9487-0f55aaa1ce0a"
+					(reference "L801")
 					(unit 1)
 				)
@@
 		(on_board yes)
 		(dnp no)
-		(property "Reference" "C1006"
+		(property "Reference" "C806"
 			(at 174.244 104.775 0)
 			(effects
@@
 		(instances
 			(project "ESP_bare_chip_test_board"
-				(path "/45b6f84a-e69b-48be-a49b-bc68872e2c15/28425a28-8968-4679-b18b-58814452f93f/a569503a-4f7e-494d-9487-0f55aaa1ce0a"
-					(reference "C1006")
+				(path "/45b6f84a-e69b-48be-a49b-bc68872e2c15/f48098a1-cacc-4192-b650-2a34a2ba76dc/1ca534e3-2263-4539-8aa0-ff724a69b5d8/a569503a-4f7e-494d-9487-0f55aaa1ce0a"
+					(reference "C806")
 					(unit 1)
 				)
@@
 		(dnp no)
 		(fields_autoplaced yes)
-		(property "Reference" "#PWR0901"
+		(property "Reference" "#PWR801"
 			(at 101.6 163.83 0)
 			(effects
@@
 		(instances
 			(project "ESP_bare_chip_test_board"
-				(path "/45b6f84a-e69b-48be-a49b-bc68872e2c15/28425a28-8968-4679-b18b-58814452f93f/a569503a-4f7e-494d-9487-0f55aaa1ce0a"
-					(reference "#PWR0901")
+				(path "/45b6f84a-e69b-48be-a49b-bc68872e2c15/f48098a1-cacc-4192-b650-2a34a2ba76dc/1ca534e3-2263-4539-8aa0-ff724a69b5d8/a569503a-4f7e-494d-9487-0f55aaa1ce0a"
+					(reference "#PWR801")
 					(unit 1)
 				)
@@
 		(on_board yes)
 		(dnp no)
-		(property "Reference" "C1005"
+		(property "Reference" "C805"
 			(at 164.084 104.775 0)
 			(effects
@@
 		(instances
 			(project "ESP_bare_chip_test_board"
-				(path "/45b6f84a-e69b-48be-a49b-bc68872e2c15/28425a28-8968-4679-b18b-58814452f93f/a569503a-4f7e-494d-9487-0f55aaa1ce0a"
-					(reference "C1005")
+				(path "/45b6f84a-e69b-48be-a49b-bc68872e2c15/f48098a1-cacc-4192-b650-2a34a2ba76dc/1ca534e3-2263-4539-8aa0-ff724a69b5d8/a569503a-4f7e-494d-9487-0f55aaa1ce0a"
+					(reference "C805")
 					(unit 1)
 				)
@@
 		(dnp no)
 		(fields_autoplaced yes)
-		(property "Reference" "#PWR01002"
+		(property "Reference" "#PWR802"
 			(at 111.76 133.35 0)
 			(effects
@@
 		(instances
 			(project "ESP_bare_chip_test_board"
-				(path "/45b6f84a-e69b-48be-a49b-bc68872e2c15/28425a28-8968-4679-b18b-58814452f93f/a569503a-4f7e-494d-9487-0f55aaa1ce0a"
-					(reference "#PWR01002")
+				(path "/45b6f84a-e69b-48be-a49b-bc68872e2c15/f48098a1-cacc-4192-b650-2a34a2ba76dc/1ca534e3-2263-4539-8aa0-ff724a69b5d8/a569503a-4f7e-494d-9487-0f55aaa1ce0a"
+					(reference "#PWR802")
 					(unit 1)
 				)
@@
 		(on_board yes)
 		(dnp no)
-		(property "Reference" "C1007"
+		(property "Reference" "C807"
 			(at 184.404 104.775 0)
 			(effects
@@
 		(instances
 			(project "ESP_bare_chip_test_board"
-				(path "/45b6f84a-e69b-48be-a49b-bc68872e2c15/28425a28-8968-4679-b18b-58814452f93f/a569503a-4f7e-494d-9487-0f55aaa1ce0a"
-					(reference "C1007")
-					(unit 1)
-				)
+				(path "/45b6f84a-e69b-48be-a49b-bc68872e2c15/f48098a1-cacc-4192-b650-2a34a2ba76dc/1ca534e3-2263-4539-8aa0-ff724a69b5d8/a569503a-4f7e-494d-9487-0f55aaa1ce0a"
+					(reference "C807")
+					(unit 1)
+				)
