File: subsheet/connector_GPIB.kicad_sch (KiCad schematic)
At the start: 1 part, among them J1201 NorComp - 112-024-113RYY1

Commit message: Move all subsheets into 'main' subsheet, below root
Keeping all the subsheets in a dedicated 'subsheet' folder makes things
much, much neater. However, specifying filepaths for subsheets has an
interesting problem; they use paths RELATIVE TO THE PARENT SHEET.

The consequence of is that if a subsheet is part of the root sheet, it
needs to be prefixed with 'subsheet/', but NOT if it's further down.
This inconsistency can be resolved by having a single 'main' sheet at
the top that doesn't move.

It's also useful to have a top-level space to put down changelogs,
descriptions etc.
Parts:
- renumbered J1201 to J1101
Changed lines of the file:
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@@
 		(shape bidirectional)
 		(at 132.08 86.36 180)
-		(fields_autoplaced yes)
 		(effects
 			(font
@@
 		(shape bidirectional)
 		(at 124.46 96.52 180)
-		(fields_autoplaced yes)
 		(effects
 			(font
@@
 		(shape bidirectional)
 		(at 152.4 104.14 0)
-		(fields_autoplaced yes)
 		(effects
 			(font
@@
 		(shape bidirectional)
 		(at 152.4 99.06 0)
-		(fields_autoplaced yes)
 		(effects
 			(font
@@
 		(shape bidirectional)
 		(at 124.46 99.06 180)
-		(fields_autoplaced yes)
 		(effects
 			(font
@@
 		(shape bidirectional)
 		(at 132.08 91.44 180)
-		(fields_autoplaced yes)
 		(effects
 			(font
@@
 		(shape bidirectional)
 		(at 124.46 104.14 180)
-		(fields_autoplaced yes)
 		(effects
 			(font
@@
 		(shape bidirectional)
 		(at 152.4 96.52 0)
-		(fields_autoplaced yes)
 		(effects
 			(font
@@
 		(shape bidirectional)
 		(at 132.08 93.98 180)
-		(fields_autoplaced yes)
 		(effects
 			(font
@@
 		(shape bidirectional)
 		(at 132.08 81.28 180)
-		(fields_autoplaced yes)
 		(effects
 			(font
@@
 		(shape bidirectional)
 		(at 132.08 83.82 180)
-		(fields_autoplaced yes)
 		(effects
 			(font
@@
 		(shape bidirectional)
 		(at 144.78 93.98 0)
-		(fields_autoplaced yes)
 		(effects
 			(font
@@
 		(shape bidirectional)
 		(at 124.46 101.6 180)
-		(fields_autoplaced yes)
 		(effects
 			(font
@@
 		(shape bidirectional)
 		(at 152.4 101.6 0)
-		(fields_autoplaced yes)
 		(effects
 			(font
@@
 		(shape bidirectional)
 		(at 132.08 88.9 180)
-		(fields_autoplaced yes)
 		(effects
 			(font
@@
 		(shape bidirectional)
 		(at 132.08 78.74 180)
-		(fields_autoplaced yes)
 		(effects
 			(font
@@
 		(on_board yes)
 		(dnp no)
-		(property "Reference" "#PWR01201"
+		(property "Reference" "#PWR1101"
 			(at 160.02 80.01 0)
 			(effects
@@
 		(instances
 			(project "ESP_bare_chip_test_board"
-				(path "/45b6f84a-e69b-48be-a49b-bc68872e2c15/3ac85730-69ac-49b3-9a57-3b8bd09542e4"
-					(reference "#PWR01201")
+				(path "/45b6f84a-e69b-48be-a49b-bc68872e2c15/f48098a1-cacc-4192-b650-2a34a2ba76dc/7ccd7424-4ed5-46cc-bfe9-7291525268e5"
+					(reference "#PWR1101")
 					(unit 1)
 				)
@@
 		(on_board yes)
 		(dnp no)
-		(property "Reference" "J1201"
+		(property "Reference" "J1101"
 			(at 138.43 109.6518 0)
 			(effects
@@
 		(instances
 			(project "ESP_bare_chip_test_board"
-				(path "/45b6f84a-e69b-48be-a49b-bc68872e2c15/3ac85730-69ac-49b3-9a57-3b8bd09542e4"
-					(reference "J1201")
+				(path "/45b6f84a-e69b-48be-a49b-bc68872e2c15/f48098a1-cacc-4192-b650-2a34a2ba76dc/7ccd7424-4ed5-46cc-bfe9-7291525268e5"
+					(reference "J1101")
 					(unit 1)
 				)
