File: subsheet/usb.kicad_sch (KiCad schematic)
At the start: 6 parts, among them J801 USB_C_Receptacle, J802 USB_C_Receptacle, U601 D1213A-04TS-7, U801 D1213A-04TS-7

Commit message: Silkscreen work. Edit tittle block/version number
Other:
- company: copyright Escape This 2024 -> (c) Vincent Dalstra
- title: Puzzle Board -> Untitled 4-layer JLCPCB
Changed lines of the file:
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@@
 	(paper "A5")
 	(title_block
-		(title "Puzzle Board")
-		(date "2024-03-20")
-		(rev "4.0.0")
-		(company "copyright Escape This 2024")
+		(title "Untitled 4-layer JLCPCB")
+		(date "2024-06-14")
+		(rev "1.0.0")
+		(company "(c) Vincent Dalstra")
 		(comment 1 "Drawn by: VGD")
 		(comment 2 "Check by:")

Commit message: Move all subsheets into 'main' subsheet, below root
Keeping all the subsheets in a dedicated 'subsheet' folder makes things
much, much neater. However, specifying filepaths for subsheets has an
interesting problem; they use paths RELATIVE TO THE PARENT SHEET.

The consequence of is that if a subsheet is part of the root sheet, it
needs to be prefixed with 'subsheet/', but NOT if it's further down.
This inconsistency can be resolved by having a single 'main' sheet at
the top that doesn't move.

It's also useful to have a top-level space to put down changelogs,
descriptions etc.
Parts:
- renumbered J801 to J1001, J802 to J1002, R601 to R1001, R602 to R1002, U801 to U1001, U601 to U1002
Changed lines of the file:
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@@
 	(label "CC1"
 		(at 5.08 76.2 0)
-		(fields_autoplaced yes)
 		(effects
 			(font
@@
 	(label "CC2"
 		(at 5.08 71.12 0)
-		(fields_autoplaced yes)
 		(effects
 			(font
@@
 	(label "CC2"
 		(at 96.52 71.12 0)
-		(fields_autoplaced yes)
 		(effects
 			(font
@@
 	(label "USB_VBUS"
 		(at 60.96 25.4 0)
-		(fields_autoplaced yes)
 		(effects
 			(font
@@
 	(label "CC2"
 		(at 43.18 45.72 0)
-		(fields_autoplaced yes)
 		(effects
 			(font
@@
 	(label "CC1"
 		(at 43.18 43.18 0)
-		(fields_autoplaced yes)
 		(effects
 			(font
@@
 	(label "CC1"
 		(at 96.52 76.2 0)
-		(fields_autoplaced yes)
 		(effects
 			(font
@@
 		(shape bidirectional)
 		(at 180.34 25.4 0)
-		(fields_autoplaced yes)
 		(effects
 			(font
@@
 		(shape bidirectional)
 		(at 116.84 99.06 0)
-		(fields_autoplaced yes)
 		(effects
 			(font
@@
 		(shape bidirectional)
 		(at 116.84 96.52 0)
-		(fields_autoplaced yes)
 		(effects
 			(font
@@
 		(shape output)
 		(at 177.8 55.88 0)
-		(fields_autoplaced yes)
 		(effects
 			(font
@@
 		(shape output)
 		(at 177.8 58.42 0)
-		(fields_autoplaced yes)
 		(effects
 			(font
@@
 		(dnp no)
 		(fields_autoplaced yes)
-		(property "Reference" "U801"
+		(property "Reference" "U1001"
 			(at -3.4289 60.96 0)
 			(effects
@@
 		(instances
 			(project "ESP_bare_chip_test_board"
-				(path "/45b6f84a-e69b-48be-a49b-bc68872e2c15/e324977a-58a1-4f1d-a668-70aacbf37a3e"
-					(reference "U801")
+				(path "/45b6f84a-e69b-48be-a49b-bc68872e2c15/f48098a1-cacc-4192-b650-2a34a2ba76dc/4d0d291b-97b9-4a0d-a83b-67ee582f6b4f"
+					(reference "U1001")
 					(unit 1)
 				)
@@
 		(dnp yes)
 		(fields_autoplaced yes)
-		(property "Reference" "J802"
+		(property "Reference" "J1002"
 			(at 27.94 30.48 0)
 			(effects
@@
 		(instances
 			(project "ESP_bare_chip_test_board"
-				(path "/45b6f84a-e69b-48be-a49b-bc68872e2c15/e324977a-58a1-4f1d-a668-70aacbf37a3e"
-					(reference "J802")
+				(path "/45b6f84a-e69b-48be-a49b-bc68872e2c15/f48098a1-cacc-4192-b650-2a34a2ba76dc/4d0d291b-97b9-4a0d-a83b-67ee582f6b4f"
+					(reference "J1002")
 					(unit 1)
 				)
@@
 		(dnp no)
 		(fields_autoplaced yes)
-		(property "Reference" "#PWR0804"
+		(property "Reference" "#PWR1004"
 			(at -5.08 90.17 0)
 			(effects
@@
 		(instances
 			(project "ESP_bare_chip_test_board"
-				(path "/45b6f84a-e69b-48be-a49b-bc68872e2c15/e324977a-58a1-4f1d-a668-70aacbf37a3e"
-					(reference "#PWR0804")
+				(path "/45b6f84a-e69b-48be-a49b-bc68872e2c15/f48098a1-cacc-4192-b650-2a34a2ba76dc/4d0d291b-97b9-4a0d-a83b-67ee582f6b4f"
+					(reference "#PWR1004")
 					(unit 1)
 				)
@@
 		(dnp no)
 		(fields_autoplaced yes)
-		(property "Reference" "R602"
+		(property "Reference" "R1002"
 			(at 167.64 66.0399 0)
 			(effects
@@
 		(instances
 			(project "ESP_bare_chip_test_board"
-				(path "/45b6f84a-e69b-48be-a49b-bc68872e2c15/e324977a-58a1-4f1d-a668-70aacbf37a3e"
-					(reference "R602")
+				(path "/45b6f84a-e69b-48be-a49b-bc68872e2c15/f48098a1-cacc-4192-b650-2a34a2ba76dc/4d0d291b-97b9-4a0d-a83b-67ee582f6b4f"
+					(reference "R1002")
 					(unit 1)
 				)
@@
 		(dnp no)
 		(fields_autoplaced yes)
-		(property "Reference" "#PWR0603"
+		(property "Reference" "#PWR1009"
 			(at 154.94 80.01 0)
 			(effects
@@
 		(instances
 			(project "ESP_bare_chip_test_board"
-				(path "/45b6f84a-e69b-48be-a49b-bc68872e2c15/e324977a-58a1-4f1d-a668-70aacbf37a3e"
-					(reference "#PWR0603")
+				(path "/45b6f84a-e69b-48be-a49b-bc68872e2c15/f48098a1-cacc-4192-b650-2a34a2ba76dc/4d0d291b-97b9-4a0d-a83b-67ee582f6b4f"
+					(reference "#PWR1009")
 					(unit 1)
 				)
@@
 		(dnp no)
 		(fields_autoplaced yes)
-		(property "Reference" "#PWR0601"
+		(property "Reference" "#PWR1007"
 			(at 86.36 39.37 0)
 			(effects
@@
 		(instances
 			(project "ESP_bare_chip_test_board"
-				(path "/45b6f84a-e69b-48be-a49b-bc68872e2c15/e324977a-58a1-4f1d-a668-70aacbf37a3e"
-					(reference "#PWR0601")
+				(path "/45b6f84a-e69b-48be-a49b-bc68872e2c15/f48098a1-cacc-4192-b650-2a34a2ba76dc/4d0d291b-97b9-4a0d-a83b-67ee582f6b4f"
+					(reference "#PWR1007")
 					(unit 1)
 				)
@@
 		(dnp yes)
 		(fields_autoplaced yes)
-		(property "Reference" "U601"
+		(property "Reference" "U1002"
 			(at 88.0111 60.96 0)
 			(effects
@@
 		(instances
 			(project "ESP_bare_chip_test_board"
-				(path "/45b6f84a-e69b-48be-a49b-bc68872e2c15/e324977a-58a1-4f1d-a668-70aacbf37a3e"
-					(reference "U601")
+				(path "/45b6f84a-e69b-48be-a49b-bc68872e2c15/f48098a1-cacc-4192-b650-2a34a2ba76dc/4d0d291b-97b9-4a0d-a83b-67ee582f6b4f"
+					(reference "U1002")
 					(unit 1)
 				)
@@
 		(dnp no)
 		(fields_autoplaced yes)
-		(property "Reference" "#PWR0801"
+		(property "Reference" "#PWR1001"
 			(at -48.26 110.49 0)
 			(effects
@@
 		(instances
 			(project "ESP_bare_chip_test_board"
-				(path "/45b6f84a-e69b-48be-a49b-bc68872e2c15/e324977a-58a1-4f1d-a668-70aacbf37a3e"
-					(reference "#PWR0801")
+				(path "/45b6f84a-e69b-48be-a49b-bc68872e2c15/f48098a1-cacc-4192-b650-2a34a2ba76dc/4d0d291b-97b9-4a0d-a83b-67ee582f6b4f"
+					(reference "#PWR1001")
 					(unit 1)
 				)
@@
 		(dnp no)
 		(fields_autoplaced yes)
-		(property "Reference" "R601"
+		(property "Reference" "R1001"
 			(at 157.48 66.0399 0)
 			(effects
@@
 		(instances
 			(project "ESP_bare_chip_test_board"
-				(path "/45b6f84a-e69b-48be-a49b-bc68872e2c15/e324977a-58a1-4f1d-a668-70aacbf37a3e"
-					(reference "R601")
+				(path "/45b6f84a-e69b-48be-a49b-bc68872e2c15/f48098a1-cacc-4192-b650-2a34a2ba76dc/4d0d291b-97b9-4a0d-a83b-67ee582f6b4f"
+					(reference "R1001")
 					(unit 1)
 				)
@@
 		(dnp no)
 		(fields_autoplaced yes)
-		(property "Reference" "#PWR0602"
+		(property "Reference" "#PWR1008"
 			(at 86.36 90.17 0)
 			(effects
@@
 		(instances
 			(project "ESP_bare_chip_test_board"
-				(path "/45b6f84a-e69b-48be-a49b-bc68872e2c15/e324977a-58a1-4f1d-a668-70aacbf37a3e"
-					(reference "#PWR0602")
+				(path "/45b6f84a-e69b-48be-a49b-bc68872e2c15/f48098a1-cacc-4192-b650-2a34a2ba76dc/4d0d291b-97b9-4a0d-a83b-67ee582f6b4f"
+					(reference "#PWR1008")
 					(unit 1)
 				)
@@
 		(dnp no)
 		(fields_autoplaced yes)
-		(property "Reference" "#PWR0604"
+		(property "Reference" "#PWR1010"
 			(at 165.1 80.01 0)
 			(effects
@@
 		(instances
 			(project "ESP_bare_chip_test_board"
-				(path "/45b6f84a-e69b-48be-a49b-bc68872e2c15/e324977a-58a1-4f1d-a668-70aacbf37a3e"
-					(reference "#PWR0604")
+				(path "/45b6f84a-e69b-48be-a49b-bc68872e2c15/f48098a1-cacc-4192-b650-2a34a2ba76dc/4d0d291b-97b9-4a0d-a83b-67ee582f6b4f"
+					(reference "#PWR1010")
 					(unit 1)
 				)
@@
 		(dnp no)
 		(fields_autoplaced yes)
-		(property "Reference" "J801"
+		(property "Reference" "J1001"
 			(at -40.64 30.48 0)
 			(effects
@@
 		(instances
 			(project "ESP_bare_chip_test_board"
-				(path "/45b6f84a-e69b-48be-a49b-bc68872e2c15/e324977a-58a1-4f1d-a668-70aacbf37a3e"
-					(reference "J801")
+				(path "/45b6f84a-e69b-48be-a49b-bc68872e2c15/f48098a1-cacc-4192-b650-2a34a2ba76dc/4d0d291b-97b9-4a0d-a83b-67ee582f6b4f"
+					(reference "J1001")
 					(unit 1)
 				)
@@
 		(dnp no)
 		(fields_autoplaced yes)
-		(property "Reference" "#FLG0601"
+		(property "Reference" "#FLG1001"
 			(at 45.72 36.195 0)
 			(effects
@@
 		(instances
 			(project "ESP_bare_chip_test_board"
-				(path "/45b6f84a-e69b-48be-a49b-bc68872e2c15/e324977a-58a1-4f1d-a668-70aacbf37a3e"
-					(reference "#FLG0601")
+				(path "/45b6f84a-e69b-48be-a49b-bc68872e2c15/f48098a1-cacc-4192-b650-2a34a2ba76dc/4d0d291b-97b9-4a0d-a83b-67ee582f6b4f"
+					(reference "#FLG1001")
 					(unit 1)
 				)
@@
 		(dnp no)
 		(fields_autoplaced yes)
-		(property "Reference" "#PWR0803"
+		(property "Reference" "#PWR1003"
 			(at -5.08 26.67 0)
 			(effects
@@
 		(instances
 			(project "ESP_bare_chip_test_board"
-				(path "/45b6f84a-e69b-48be-a49b-bc68872e2c15/e324977a-58a1-4f1d-a668-70aacbf37a3e"
-					(reference "#PWR0803")
+				(path "/45b6f84a-e69b-48be-a49b-bc68872e2c15/f48098a1-cacc-4192-b650-2a34a2ba76dc/4d0d291b-97b9-4a0d-a83b-67ee582f6b4f"
+					(reference "#PWR1003")
 					(unit 1)
 				)
@@
 		(dnp no)
 		(fields_autoplaced yes)
-		(property "Reference" "#PWR0802"
+		(property "Reference" "#PWR1002"
 			(at -40.64 110.49 0)
 			(effects
@@
 		(instances
 			(project "ESP_bare_chip_test_board"
-				(path "/45b6f84a-e69b-48be-a49b-bc68872e2c15/e324977a-58a1-4f1d-a668-70aacbf37a3e"
-					(reference "#PWR0802")
+				(path "/45b6f84a-e69b-48be-a49b-bc68872e2c15/f48098a1-cacc-4192-b650-2a34a2ba76dc/4d0d291b-97b9-4a0d-a83b-67ee582f6b4f"
+					(reference "#PWR1002")
 					(unit 1)
 				)
@@
 		(dnp no)
 		(fields_autoplaced yes)
-		(property "Reference" "#PWR0806"
+		(property "Reference" "#PWR1006"
 			(at 27.94 110.49 0)
 			(effects
@@
 		(instances
 			(project "ESP_bare_chip_test_board"
-				(path "/45b6f84a-e69b-48be-a49b-bc68872e2c15/e324977a-58a1-4f1d-a668-70aacbf37a3e"
-					(reference "#PWR0806")
+				(path "/45b6f84a-e69b-48be-a49b-bc68872e2c15/f48098a1-cacc-4192-b650-2a34a2ba76dc/4d0d291b-97b9-4a0d-a83b-67ee582f6b4f"
+					(reference "#PWR1006")
 					(unit 1)
 				)
@@
 		(dnp no)
 		(fields_autoplaced yes)
-		(property "Reference" "#PWR0805"
+		(property "Reference" "#PWR1005"
 			(at 20.32 110.49 0)
 			(effects
@@
 		(instances
 			(project "ESP_bare_chip_test_board"
-				(path "/45b6f84a-e69b-48be-a49b-bc68872e2c15/e324977a-58a1-4f1d-a668-70aacbf37a3e"
-					(reference "#PWR0805")
-					(unit 1)
-				)
+				(path "/45b6f84a-e69b-48be-a49b-bc68872e2c15/f48098a1-cacc-4192-b650-2a34a2ba76dc/4d0d291b-97b9-4a0d-a83b-67ee582f6b4f"
+					(reference "#PWR1005")
+					(unit 1)
+				)
